Commit message: Fixing lane detector

File: src/robot_simulation/mentorpi_sim/urdf/ack.urdf.xacro (robot description, xacro)
@@ -1,25 +1,4 @@
 <?xml version="1.0" ?>
 <robot name="ack" xmlns:xacro="http://ros.org/wiki/xacro">
-  <gazebo reference="depth_cam">
-    <sensor type="camera" name="front_camera">
-      <update_rate>30.0</update_rate>
-      <camera>
-        <horizontal_fov>1.3962634</horizontal_fov>
-        <image>
-          <width>640</width>
-          <height>480</height>
-          <format>R8G8B8</format>
-        </image>
-        <clip>
-          <near>0.02</near>
-          <far>300</far>
-        </clip>
-      </camera>
-      <topic>/camera/image_raw</topic>
-      <plugin filename="ignition-gazebo-sensors-system" name="ignition::gazebo::systems::Sensors">
-        <render_engine>ogre2</render_engine>
-      </plugin>
-    </sensor>
-  </gazebo>
   <gazebo>
     <plugin filename="ignition-gazebo-diff-drive-system" name="ignition::gazebo::systems::DiffDrive">
@@ -34,27 +13,18 @@
     </plugin>
   </gazebo>
-  <material name="black">
-    <color rgba="0 0 0 1"/>
-  </material>
+  <material name="black"><color rgba="0.1 0.1 0.1 1"/></material>
+  <material name="blue"><color rgba="0.0 0.4 1.0 1"/></material>
   <link name="base_link">
     <inertial>
-      <origin rpy="0 0 0" xyz="-0.00186669751054189 3.0253386351986E-05 -0.00605296088229322"/>
-      <mass value="0.0961047465616957"/>
-      <inertia ixx="8.55867486364231E-05" ixy="3.41346959938296E-08" ixz="1.64755227278164E-05" iyy="0.000277248181555496" iyz="-2.95282759133104E-08" izz="0.000344246448853775"/>
+      <origin rpy="0 0 0" xyz="-0.001 0 -0.006"/>
+      <mass value="0.5"/>
+      <inertia ixx="0.001" ixy="0" ixz="0" iyy="0.001" iyz="0" izz="0.001"/>
     </inertial>
     <visual>
-      <origin rpy="0 0 0" xyz="0 0 0"/>
-      <geometry>
-        <mesh filename="file://$(find mentorpi_sim)/meshes/acker/base_link.stl"/>
-      </geometry>
-      <material name="">
-        <color rgba="1 1 1 1"/>
-      </material>
+      <geometry><box size="0.2 0.12 0.05"/></geometry>
+      <material name="blue"/>
     </visual>
     <collision>
-      <origin rpy="0 0 0" xyz="0 0 0"/>
-      <geometry>
-        <mesh filename="file://$(find mentorpi_sim)/meshes/acker/base_link.stl"/>
-      </geometry>
+      <geometry><box size="0.2 0.12 0.05"/></geometry>
     </collision>
   </link>
@@ -65,129 +35,65 @@
     <origin xyz="0 0 0.07" rpy="0 0 0"/>
   </joint>
-  <link name="wheel_lf_Link">
+  <xacro:macro name="wheel" params="prefix x y">
+    <link name="wheel_${prefix}_Link">
+      <visual>
+        <origin rpy="1.5708 0 0" xyz="0 0 0"/>
+        <geometry><cylinder radius="0.033" length="0.02"/></geometry>
+        <material name="black"/>
+      </visual>
+      <collision>
+        <origin rpy="1.5708 0 0" xyz="0 0 0"/>
+        <geometry><cylinder radius="0.033" length="0.02"/></geometry>
+      </collision>
+      <inertial>
+        <mass value="0.05"/>
+        <inertia ixx="0.0001" ixy="0" ixz="0" iyy="0.0001" iyz="0" izz="0.0001"/>
+      </inertial>
+    </link>
+    <joint name="wheel_${prefix}_Joint" type="continuous">
+      <origin rpy="0 0 0" xyz="${x} ${y} -0.028"/>
+      <parent link="base_link"/>
+      <child link="wheel_${prefix}_Link"/>
+      <axis xyz="0 1 0"/>
+    </joint>
+  </xacro:macro>
+  <xacro:wheel prefix="lf" x="0.07" y="0.07"/>
+  <xacro:wheel prefix="rf" x="0.07" y="-0.07"/>
+  <xacro:wheel prefix="lb" x="-0.07" y="0.07"/>
+  <xacro:wheel prefix="rb" x="-0.07" y="-0.07"/>
+  <link name="depth_cam">
+    <visual>
+      <geometry><box size="0.02 0.05 0.05"/></geometry>
+      <material name="red"/>
+    </visual>
     <inertial>
-      <origin rpy="0 0 0" xyz="1.65897579444685E-06 -0.00270913022688685 -1.5546673051009E-06"/>
-      <mass value="0.0252873083503169"/>
-      <inertia ixx="1.00371783485335E-05" ixy="4.93900109379125E-11" ixz="7.42104604492639E-10" iyy="1.67620175120314E-05" iyz="-5.47583950457701E-11" izz="1.00370342405297E-05"/>
+      <mass value="0.01"/>
+      <inertia ixx="0.0001" ixy="0" ixz="0" iyy="0.0001" iyz="0" izz="0.0001"/>
     </inertial>
-    <visual>
-      <origin rpy="0 0 0" xyz="0 0 0"/>
-      <geometry>
-        <mesh filename="file://$(find mentorpi_sim)/meshes/acker/wheel_lf_Link.stl"/>
-      </geometry>
-    </visual>
-    <collision>
-      <origin rpy="0 0 0" xyz="0 0 0"/>
-      <geometry>
-        <mesh filename="file://$(find mentorpi_sim)/meshes/acker/wheel_lf_Link.stl"/>
-      </geometry>
-    </collision>
-  </link>
-  <joint name="wheel_lf_Joint" type="continuous">
-    <origin rpy="0 0 0" xyz="0.06679 0.069739 -0.0288"/>
-    <parent link="base_link"/>
-    <child link="wheel_lf_Link"/>
-    <axis xyz="-2.2918E-05 1 1.9551E-05"/>
-  </joint>
-  <link name="wheel_rf_Link">
-    <inertial>
-      <origin rpy="0 0 0" xyz="-1.48986965733955E-06 0.0027090575018239 1.16299057125596E-06"/>
-      <mass value="0.0252873548617242"/>
-      <inertia ixx="1.00360241846408E-05" ixy="-5.83065201444192E-11" ixz="-8.3023958781985E-11" iyy="1.67622954977732E-05" iyz="6.31638512668579E-11" izz="1.00384960556047E-05"/>
-    </inertial>
-    <visual>
-      <origin rpy="0 0 0" xyz="0 0 0"/>
-      <geometry>
-        <mesh filename="file://$(find mentorpi_sim)/meshes/acker/wheel_rf_Link.stl"/>
-      </geometry>
-    </visual>
-    <collision>
-      <origin rpy="0 0 0" xyz="0 0 0"/>
-      <geometry>
-        <mesh filename="file://$(find mentorpi_sim)/meshes/acker/wheel_rf_Link.stl"/>
-      </geometry>
-    </collision>
-  </link>
-  <joint name="wheel_rf_Joint" type="continuous">
-    <origin rpy="0 0 0" xyz="0.066794 -0.069739 -0.028803"/>
-    <parent link="base_link"/>
-    <child link="wheel_rf_Link"/>
-    <axis xyz="-2.2918E-05 1 1.9551E-05"/>
-  </joint>
-  <link name="wheel_lb_Link">
-    <inertial>
-      <origin rpy="0 0 0" xyz="1.62806317080544E-06 -0.00317716794378092 -1.54238045318306E-06"/>
-      <mass value="0.0271078161230754"/>
-      <inertia ixx="1.01056035703468E-05" ixy="4.60479373806495E-11" ixz="7.43896782806142E-10" iyy="1.67990600599721E-05" iyz="-5.763890541079E-11" izz="1.01072652738793E-05"/>
-    </inertial>
-    <visual>
-      <origin rpy="0 0 0" xyz="0 0 0"/>
-      <geometry>
-        <mesh filename="file://$(find mentorpi_sim)/meshes/acker/wheel_lb_Link.stl"/>
-      </geometry>
-    </visual>
-    <collision>
-      <origin rpy="0 0 0" xyz="0 0 0"/>
-      <geometry>
-        <mesh filename="file://$(find mentorpi_sim)/meshes/acker/wheel_lb_Link.stl"/>
-      </geometry>
-    </collision>
-  </link>
-  <joint name="wheel_lb_Joint" type="continuous">
-    <origin rpy="0 0 0" xyz="-0.070313 0.07014 -0.027793"/>
-    <parent link="base_link"/>
-    <child link="wheel_lb_Link"/>
-    <axis xyz="-2.2787E-05 1 1.9439E-05"/>
-  </joint>
-  <link name="wheel_rb_Link">
-    <inertial>
-      <origin rpy="0 0 0" xyz="-1.50804700475154E-06 0.00317707027691583 1.18963606317302E-06"/>
-      <mass value="0.0271078005024283"/>
-      <inertia ixx="1.01044417409685E-05" ixy="-5.83069005452564E-11" ixz="-7.56886841840775E-11" iyy="1.67993271276785E-05" iyz="6.31638424138502E-11" izz="1.01087182681654E-05"/>
-    </inertial>
-    <visual>
-      <origin rpy="0 0 0" xyz="0 0 0"/>
-      <geometry>
-        <mesh filename="file://$(find mentorpi_sim)/meshes/acker/wheel_rb_Link.stl"/>
-      </geometry>
-    </visual>
-    <collision>
-      <origin rpy="0 0 0" xyz="0 0 0"/>
-      <geometry>
-        <mesh filename="file://$(find mentorpi_sim)/meshes/acker/wheel_rb_Link.stl"/>
-      </geometry>
-    </collision>
-  </link>
-  <joint name="wheel_rb_Joint" type="continuous">
-    <origin rpy="0 0 0" xyz="-0.07031 -0.07014 -0.027796"/>
-    <parent link="base_link"/>
-    <child link="wheel_rb_Link"/>
-    <axis xyz="-2.2787E-05 1 1.9439E-05"/>
-  </joint>
-  <link name="depth_cam">
-    <inertial>
-      <origin rpy="0 0 0" xyz="0.0023402290651429 0.00113784597946548 -0.0102127064032341"/>
-      <mass value="0.0270474748429678"/>
-      <inertia ixx="1.43718505822118E-05" ixy="1.24779382573379E-07" ixz="1.29836477956744E-08" iyy="1.65912768209848E-06" iyz="2.28291478579102E-08" izz="1.45615925510082E-05"/>
-    </inertial>
-    <visual>
-      <origin rpy="0 0 0" xyz="0 0 0"/>
-      <geometry>
-        <box size="0.02 0.05 0.05"/>
-      </geometry>
-      <material name=""><color rgba="0 0 1 1"/></material>
-    </visual>
-    <collision>
-      <origin rpy="0 0 0" xyz="0 0 0"/>
-      <geometry>
-        <box size="0.02 0.05 0.05"/>
-      </geometry>
-    </collision>
   </link>
   <joint name="cam_Joint" type="fixed">
-    <origin rpy="0 0 0" xyz="0.064015 -0.00013463 0.051155"/>
+    <origin rpy="0 0 0" xyz="0.1 0 0.04"/>
     <parent link="base_link"/>
     <child link="depth_cam"/>
-    <axis xyz="0 0 0"/>
   </joint>
+  <gazebo reference="depth_cam">
+    <sensor name="front_camera" type="camera">
+      <camera>
+        <horizontal_fov>1.396</horizontal_fov>
+        <image>
+          <width>640</width>
+          <height>480</height>
+          <format>R8G8B8</format>
+        </image>
+        <clip>
+          <near>0.02</near>
+          <far>100.0</far>
+        </clip>
+      </camera>
+      <always_on>1</always_on>
+      <update_rate>30</update_rate>
+      <visualize>true</visualize>
+      <topic>/camera/image_raw</topic>
+    </sensor>
+  </gazebo>
 </robot>
